File: epoch_program_adapter.sch (KiCad schematic (older format))
At the start: 8 parts, among them J1 CONN_02X05, J2 CONN_01X05, Q1 DMP1045U, U1 LTC4412

Commit message: Increase drill size to 2.1.  Rework daughter board
Parts:
- removed H1, H2: MH2mm, my-fp-library:MH2mm, symbol MH2mm
- added H1, H2: MH2mm, my-fp-library:MH2.1mm, symbol MH2.1mm
Connections:
- net labels added: +3.3V
- net labels removed: (+3.3V), GND, VCC
- wire segments 30 -> 31
Changed lines of the file:
@@
 LIBS:marks
 LIBS:epoch_program_adapter-cache
-LIBS:epoch-cache
 EELAYER 25 0
 EELAYER END
@@
 	1    0    0    -1
 $EndComp
-$Comp
-L VCC #PWR5
-U 1 1 59186FBD
-P 6950 2800
-F 0 "#PWR5" H 6950 2900 30  0001 C CNN
-F 1 "VCC" H 6950 2900 30  0000 C CNN
-F 2 "" H 6950 2800 60  0000 C CNN
-F 3 "" H 6950 2800 60  0000 C CNN
-	1    6950 2800
-	1    0    0    -1
-$EndComp
-$Comp
-L GND #PWR4
-U 1 1 591871C3
-P 6750 3400
-F 0 "#PWR4" H 6750 3400 30  0001 C CNN
-F 1 "GND" H 6750 3330 30  0001 C CNN
-F 2 "" H 6750 3400 60  0000 C CNN
-F 3 "" H 6750 3400 60  0000 C CNN
-	1    6750 3400
-	1    0    0    -1
-$EndComp
 Text GLabel 7650 2900 2    60   Input ~ 0
 SWDIO/+3.3V(REGUL)
@@
 Text GLabel 7300 4000 2    60   Input ~ 0
 SWDIO/+3.3V(REGUL)
-$Comp
-L VCC #PWR7
-U 1 1 591877E8
-P 7250 3700
-F 0 "#PWR7" H 7250 3800 30  0001 C CNN
-F 1 "VCC" H 7250 3800 30  0000 C CNN
-F 2 "" H 7250 3700 60  0000 C CNN
-F 3 "" H 7250 3700 60  0000 C CNN
-	1    7250 3700
-	1    0    0    -1
-$EndComp
-$Comp
-L GND #PWR6
-U 1 1 59187851
-P 7200 4500
-F 0 "#PWR6" H 7200 4500 30  0001 C CNN
-F 1 "GND" H 7200 4430 30  0001 C CNN
-F 2 "" H 7200 4500 60  0000 C CNN
-F 3 "" H 7200 4500 60  0000 C CNN
-	1    7200 4500
-	1    0    0    -1
-$EndComp
 Text GLabel 7300 4100 2    60   Input ~ 0
 SWDCLK/+3.3V(BATT)
@@
 RESET
 Wire Wire Line
-	7050 2900 6950 2900
-Wire Wire Line
-	6950 2900 6950 2800
+	6950 2900 7050 2900
+Wire Wire Line
+	6950 2600 6950 2900
 Wire Wire Line
 	7050 3000 6750 3000
@@
 Connection ~ 4850 3000
 $Comp
-L (GND) #PWR2
+L (GND) #PWR01
 U 1 1 59C6B7D4
 P 4850 4300
-F 0 "#PWR2" H 4850 4300 30  0001 C CNN
+F 0 "#PWR01" H 4850 4300 30  0001 C CNN
 F 1 "(GND)" H 4850 4300 30  0001 C CNN
 F 2 "" H 4850 4300 60  0000 C CNN
@@
 	5300 2450 5300 3700
 $Comp
-L (GND) #PWR1
+L (GND) #PWR02
 U 1 1 59C6B7D7
 P 4350 4300
-F 0 "#PWR1" H 4350 4300 30  0001 C CNN
+F 0 "#PWR02" H 4350 4300 30  0001 C CNN
 F 1 "(GND)" H 4350 4300 30  0001 C CNN
 F 2 "" H 4350 4300 60  0000 C CNN
@@
 $EndComp
 $Comp
-L (GND) #PWR3
+L (GND) #PWR03
 U 1 1 59C6B7D9
 P 6050 3550
-F 0 "#PWR3" H 6050 3550 30  0001 C CNN
+F 0 "#PWR03" H 6050 3550 30  0001 C CNN
 F 1 "(GND)" H 6050 3550 30  0001 C CNN
 F 2 "" H 6050 3550 60  0000 C CNN
@@
 Wire Wire Line
 	4600 3000 5350 3000
-Text GLabel 6200 3000 2    60   Output ~ 0
-(+3.3V)
 $Comp
 L D_Schottky D1
@@
 $EndComp
 Connection ~ 5300 2450
-$Comp
-L MH2mm H1
-U 1 1 59C6B58B
-P 9500 3100
-F 0 "H1" H 9600 3100 60  0001 C CNN
-F 1 "MH2mm" H 9500 3400 60  0001 C CNN
-F 2 "my-fp-library:MH2mm" H 9500 3100 60  0001 C CNN
-F 3 "" H 9500 3100 60  0001 C CNN
-	1    9500 3100
-	1    0    0    -1
-$EndComp
-$Comp
-L MH2mm H2
-U 1 1 59C6B5A3
-P 9500 3250
-F 0 "H2" H 9600 3250 60  0001 C CNN
-F 1 "MH2mm" H 9500 3550 60  0001 C CNN
-F 2 "my-fp-library:MH2mm" H 9500 3250 60  0001 C CNN
-F 3 "" H 9500 3250 60  0001 C CNN
-	1    9500 3250
-	1    0    0    -1
-$EndComp
-Wire Wire Line
-	5750 3000 6200 3000
+Wire Wire Line
+	5750 3000 6350 3000
 Text GLabel 4600 2450 0    60   Input ~ 0
 SWDIO/+3.3V(REGUL)
 Text GLabel 4600 3000 0    60   Input ~ 0
 SWDCLK/+3.3V(BATT)
+$Comp
+L +3.3V #PWR04
+U 1 1 59C824F8
+P 6950 2600
+F 0 "#PWR04" H 6950 2450 50  0001 C CNN
+F 1 "+3.3V" H 6950 2740 50  0000 C CNN
+F 2 "" H 6950 2600 50  0001 C CNN
+F 3 "" H 6950 2600 50  0001 C CNN
+	1    6950 2600
+	1    0    0    -1
+$EndComp
+$Comp
+L +3.3V #PWR05
+U 1 1 59C8251C
+P 7250 3700
+F 0 "#PWR05" H 7250 3550 50  0001 C CNN
+F 1 "+3.3V" H 7250 3840 50  0000 C CNN
+F 2 "" H 7250 3700 50  0001 C CNN
+F 3 "" H 7250 3700 50  0001 C CNN
+	1    7250 3700
+	1    0    0    -1
+$EndComp
+$Comp
+L +3.3V #PWR06
+U 1 1 59C82640
+P 6350 2950
+F 0 "#PWR06" H 6350 2800 50  0001 C CNN
+F 1 "+3.3V" H 6350 3090 50  0000 C CNN
+F 2 "" H 6350 2950 50  0001 C CNN
+F 3 "" H 6350 2950 50  0001 C CNN
+	1    6350 2950
+	1    0    0    -1
+$EndComp
+Wire Wire Line
+	6350 3000 6350 2950
+$Comp
+L (GND) #PWR07
+U 1 1 59C8290D
+P 7200 4500
+F 0 "#PWR07" H 7200 4500 30  0001 C CNN
+F 1 "(GND)" H 7200 4500 30  0001 C CNN
+F 2 "" H 7200 4500 60  0000 C CNN
+F 3 "" H 7200 4500 60  0000 C CNN
+	1    7200 4500
+	1    0    0    -1
+$EndComp
+$Comp
+L (GND) #PWR08
+U 1 1 59C8292A
+P 6750 3400
+F 0 "#PWR08" H 6750 3400 30  0001 C CNN
+F 1 "(GND)" H 6750 3400 30  0001 C CNN
+F 2 "" H 6750 3400 60  0000 C CNN
+F 3 "" H 6750 3400 60  0000 C CNN
+	1    6750 3400
+	1    0    0    -1
+$EndComp
+$Comp
+L MH2.1mm H1
+U 1 1 59C82B2C
+P 9350 2450
+F 0 "H1" H 9450 2450 60  0001 C CNN
+F 1 "MH2mm" H 9350 2750 60  0001 C CNN
+F 2 "my-fp-library:MH2.1mm" H 9350 2450 60  0001 C CNN
+F 3 "" H 9350 2450 60  0001 C CNN
+	1    9350 2450
+	1    0    0    -1
+$EndComp
+$Comp
+L MH2.1mm H2
+U 1 1 59C82B4C
+P 9350 2700
+F 0 "H2" H 9450 2700 60  0001 C CNN
+F 1 "MH2mm" H 9350 3000 60  0001 C CNN
+F 2 "my-fp-library:MH2.1mm" H 9350 2700 60  0001 C CNN
+F 3 "" H 9350 2700 60  0001 C CNN
+	1    9350 2700
+	1    0    0    -1
+$EndComp
 $EndSCHEMATC

Commit message: V3
Parts:
- added J3: CONN_01X02, Pin_Headers:Pin_Header_Straight_1x02_Pitch1.27mm, symbol CONN_01X02
Connections:
- net SWDCLK/+3.3V(BATT) renamed +3.3V(BATT)
- net +3.3V(BATT): now also J3.2 (P2); no longer J1.4 (P4), J2.3 (P3)
- net SWDIO/+3.3V(REGUL) renamed +3.3V(REGUL)
- net +3.3V(REGUL): now also J3.1 (P1); no longer J1.2 (P2), J2.4 (P4)
- new net SWDCLK: J1.4 (P4), J2.3 (P3)
- new net SWDIO: J1.2 (P2), J2.4 (P4)
Changed lines of the file:
@@
 $EndComp
 Text GLabel 7650 2900 2    60   Input ~ 0
-SWDIO/+3.3V(REGUL)
+SWDIO
 Text GLabel 7650 3000 2    60   Input ~ 0
-SWDCLK/+3.3V(BATT)
+SWDCLK
 Text GLabel 7650 3300 2    60   Input ~ 0
 RESET
@@
 $EndComp
 Text GLabel 7300 4000 2    60   Input ~ 0
-SWDIO/+3.3V(REGUL)
+SWDIO
 Text GLabel 7300 4100 2    60   Input ~ 0
-SWDCLK/+3.3V(BATT)
+SWDCLK
 Text GLabel 7300 4200 2    60   Input ~ 0
 RESET
@@
 	5750 3000 6350 3000
 Text GLabel 4600 2450 0    60   Input ~ 0
-SWDIO/+3.3V(REGUL)
++3.3V(REGUL)
 Text GLabel 4600 3000 0    60   Input ~ 0
-SWDCLK/+3.3V(BATT)
++3.3V(BATT)
 $Comp
 L +3.3V #PWR04
@@
 	1    0    0    -1
 $EndComp
+$Comp
+L CONN_01X02 J3
+U 1 1 5A087BD5
+P 6900 5050
+F 0 "J3" H 6900 5200 50  0000 C CNN
+F 1 "CONN_01X02" V 7000 5050 50  0000 C CNN
+F 2 "Pin_Headers:Pin_Header_Straight_1x02_Pitch1.27mm" H 6900 5050 50  0001 C CNN
+F 3 "" H 6900 5050 50  0001 C CNN
+	1    6900 5050
+	-1   0    0    1
+$EndComp
+Text GLabel 7200 5100 2    60   Input ~ 0
++3.3V(REGUL)
+Text GLabel 7200 4950 2    60   Input ~ 0
++3.3V(BATT)
+Wire Wire Line
+	7100 5000 7150 5000
+Wire Wire Line
+	7150 5000 7150 4950
+Wire Wire Line
+	7150 4950 7200 4950
+Wire Wire Line
+	7100 5100 7200 5100
 $EndSCHEMATC
