File: epoch.kicad_pcb (KiCad board)
At the start: 4 copper layers, 28 x 34 mm, 34 parts, among them J1 USB_OTG, J2 CONN_01X05, J3 CONN_01X02, P3 CONN_01X10, SW1 SW_Reset, SW2 SW_Up, SW3 SW_Middle, SW4 SW_Down, U1 MIC5219-3.3BM5, U2 ATSAMD21Ennc-AU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

Commit message: Update PCB to move battery and USB
Parts:
- moved BT1 1.66 mm to (114.8, 71.2)
Routing:
- net SWDIO: track 20.7 -> 32.7 mm, vias 2 -> 3
- net SWDCLK: track 20.5 -> 31.2 mm
- net +3.3V(BATT): track 13.8 -> 8.72 mm
- net SCL: track 31.5 -> 34.2 mm
- net EXTMODE: track 17.8 -> 15.2 mm
- net 32KHz: track 28.4 -> 29.5 mm
- net Net-(R5-Pad2): track 37.7 -> 36.8 mm
- net (GND): track 36.2 -> 37.0 mm, vias 13 -> 14
